Commit message: Robot description is finished

File: urdf/Pet/robot.xacro (robot description, xacro)
@@ -1,7 +1,7 @@
 <?xml version="1.0"?>
 <robot xmlns:xacro="http://www.ros.org/wiki/xacro" name="robot_xacro">
-<xacro:include filename="$(find exp_assignment2)/urdf/robot.gazebo"/>
+<xacro:include filename="$(find exp_assignment3)/urdf/Pet/robot.gazebo"/>
 	<xacro:property name="length_wheel" value="0.05" />
-	<xacro:property name="radius_wheel" value="0.2" />
+	<xacro:property name="radius_wheel" value="0.10" />
 	<xacro:macro name="default_inertial" params="mass">
                <inertial>
@@ -57,5 +57,5 @@
       <origin rpy="0 0 0" xyz="0 0 0"/>
       <geometry>
-        <box size="0.4 0.4 0.4"/>
+        <box size="0.3 0.3 0.3"/>
       </geometry>
       <material name="blue"/>
@@ -63,5 +63,5 @@
     <!-- caster front -->
     <collision name="caster_front_collision">
-      <origin rpy=" 0 0 0" xyz="0.15 0 -0.25"/>
+      <origin rpy=" 0 0 0" xyz="0.1 0 -0.20"/>
       <geometry>
         <sphere radius="0.05"/>
@@ -69,5 +69,5 @@
     </collision>
     <visual name="caster_front_visual">
-      <origin rpy=" 0 0 0" xyz="0.15 0 -0.25"/>
+      <origin rpy=" 0 0 0" xyz="0.1 0 -0.20"/>
       <geometry>
         <sphere radius="0.05"/>
@@ -76,5 +76,5 @@
     <!-- caster back -->
     <collision name="caster_back_collision">
-      <origin rpy=" 0 0 0" xyz="-0.15 0 -0.25"/>
+      <origin rpy=" 0 0 0" xyz="-0.1 0 -0.20"/>
       <geometry>
         <sphere radius="0.05"/>
@@ -82,7 +82,33 @@
     </collision>
     <visual name="caster_back_visual">
-      <origin rpy=" 0 0 0" xyz="-0.15 0 -0.25"/>
-      <geometry>
-        <sphere radius="0.05"/>
+      <origin rpy=" 0 0 0" xyz="-0.1 0 -0.20"/>
+      <geometry>
+        <sphere radius="0.05"/>
+      </geometry>
+    </visual>
+   <!-- arm left -->
+    <collision name="caster_back_collision">
+      <origin rpy=" 0 0 0" xyz="0.1 -0.20 0.05"/>
+      <geometry>
+        <box size="0.2 0.05 0.05"/>
+      </geometry>
+    </collision>
+    <visual name="caster_back_visual">
+      <origin rpy=" 0 0 0" xyz="0.1 -0.20 0.05"/>
+      <geometry>
+        <box size="0.2 0.05 0.05"/>
+      </geometry>
+    </visual>
+   <!-- arm left -->
+    <collision name="caster_back_collision">
+      <origin rpy=" 0 0 0" xyz="0.1 0.20 0.05"/>
+      <geometry>
+        <box size="0.2 0.05 0.05"/>
+      </geometry>
+    </collision>
+    <visual name="caster_back_visual">
+      <origin rpy=" 0 0 0" xyz="0.1 0.20 0.05"/>
+      <geometry>
+        <box size="0.2 0.05 0.05"/>
       </geometry>
     </visual>
@@ -113,5 +139,5 @@
   </link>
   <joint name="joint_right_wheel" type="continuous">
-    <origin rpy="0 0 0" xyz="0 0.275 -0.10"/>
+    <origin rpy="0 0 0" xyz="0 0.175 -0.15"/>
     <child link="link_right_wheel"/>
     <parent link="link_chassis"/>
@@ -121,5 +147,5 @@
   </joint>
   <joint name="joint_left_wheel" type="continuous">
-    <origin rpy="0 0 0" xyz="0 -0.275 -0.10"/>
+    <origin rpy="0 0 0" xyz="0 -0.175 -0.15"/>
     <child link="link_left_wheel"/>
     <parent link="link_chassis"/>
@@ -130,5 +156,5 @@
   <link name="neck_link">
 	    <collision>
-	      <origin xyz="0 0 0.30" rpy="0 0 0"/>
+	      <origin xyz="0 0 0.10" rpy="0 0 0"/>
 	      <geometry>
 		<box size="0.10 0.10 0.20"/>
@@ -136,5 +162,5 @@
 	    </collision>
 	    <visual>
-	      <origin xyz="0 0 0.30" rpy="0 0 0"/>
+	      <origin xyz="0 0 0.10" rpy="0 0 0"/>
 	      <geometry>
 		<box size="0.10 0.10 0.20"/>
@@ -158,5 +184,5 @@
 	      <origin xyz="-0.2 0 0.05" rpy="0 0 0"/>
 	      <geometry>
-		<box size="0.25 0.3 0.15"/>
+		<box size="0.10 0.20 0.1"/>
 	      </geometry>
 	    </collision>
@@ -164,5 +190,5 @@
 	      <origin xyz="-0.2 0 0.05" rpy="0 0 0"/>
 	      <geometry>
-		<box size="0.25 0.3 0.15"/>
+		<box size="0.20 0.25 0.1"/>
 	      </geometry>
 	      <material name="green"/>
@@ -176,17 +202,36 @@
   <joint name="camera_joint" type="fixed">
 	    <axis xyz="1 0 0" />
-	    <origin xyz="0.25 0 0.30" rpy="0 0 0"/>
+	    <origin xyz="0.25 0 0.185" rpy="0 0 0"/>
 	    <parent link="neck_link"/>
 	    <child link="camera_link"/>
    </joint>
-<transmission name="camera_joint_trans">
-	<type>transmission_interface/SimpleTransmission</type>
-	<joint name="camera_joint">
-		<hardwareInterface>hardware_interface/VelocityJointInterface</hardwareInterface>
-	</joint>
-	<actuator name="motor1">
-		<hardwareInterface>hardware_interface/VelocityJointInterface</hardwareInterface>
-		<mechanicalInterface>1</mechanicalInterface>
-	</actuator>
-</transmission>
+   <!-- Hokuyo sensor -->
+   <link name="hokuyo_link">
+	    <collision>
+	      <origin xyz="0 0 0.025" rpy="0 0 0"/>
+	      <geometry>
+		<box size="0.05 0.05 0.05"/>
+	      </geometry>
+	    </collision>
+	    <visual>
+	      <origin xyz="0 0 0.025" rpy="0 0 0"/>
+	      <geometry>
+		<box size="0.05 0.05 0.05"/>
+	      </geometry>
+	      <material name="red">
+		<color rgba="1 0 0 1"/>
+	      </material>
+	    </visual>
+	    <inertial>
+	      <mass value="1e-5" />
+	      <origin xyz="0 0 0" rpy="0 0 0"/>
+	      <inertia ixx="1e-6" ixy="0" ixz="0" iyy="1e-6" iyz="0" izz="1e-6" />
+	    </inertial>
+  </link>
+  <joint name="hokuyo_joint" type="fixed">
+	    <axis xyz="0 1 0" />
+	    <origin xyz="0.15 0 0.10" rpy="0 0 0"/>
+	    <parent link="link_chassis"/>
+	    <child link="hokuyo_link"/>
+  </joint>
 </robot>

Commit message: Implementation of move_base for move to point feature

File: urdf/Pet/robot.xacro (robot description, xacro)
@@ -40,9 +40,9 @@
     <color rgba="1.0 1.0 1.0 1.0"/>
   </material>
-	  <link name="link_chassis">
+    <link name="link_chassis">
     <!-- pose and inertial -->
     <pose>0 0 0.1 0 0 0</pose>
     <inertial>
-      <mass value="5"/>
+      <mass value="10"/>
       <origin rpy="0 0 0" xyz="0 0 0.1"/>
       <inertia ixx="0.0395416666667" ixy="0" ixz="0" iyy="0.106208333333" iyz="0" izz="0.106208333333"/>
@@ -61,32 +61,6 @@
       <material name="blue"/>
     </visual>
-    <!-- caster front -->
-    <collision name="caster_front_collision">
-      <origin rpy=" 0 0 0" xyz="0.1 0 -0.20"/>
-      <geometry>
-        <sphere radius="0.05"/>
-      </geometry>
-    </collision>
-    <visual name="caster_front_visual">
-      <origin rpy=" 0 0 0" xyz="0.1 0 -0.20"/>
-      <geometry>
-        <sphere radius="0.05"/>
-      </geometry>
-    </visual>
-    <!-- caster back -->
-    <collision name="caster_back_collision">
-      <origin rpy=" 0 0 0" xyz="-0.1 0 -0.20"/>
-      <geometry>
-        <sphere radius="0.05"/>
-      </geometry>
-    </collision>
-    <visual name="caster_back_visual">
-      <origin rpy=" 0 0 0" xyz="-0.1 0 -0.20"/>
-      <geometry>
-        <sphere radius="0.05"/>
-      </geometry>
-    </visual>
    <!-- arm left -->
-    <collision name="caster_back_collision">
+    <collision name="arm_left_collision">
       <origin rpy=" 0 0 0" xyz="0.1 -0.20 0.05"/>
       <geometry>
@@ -94,5 +68,5 @@
       </geometry>
     </collision>
-    <visual name="caster_back_visual">
+    <visual name="arm_left_visual">
       <origin rpy=" 0 0 0" xyz="0.1 -0.20 0.05"/>
       <geometry>
@@ -100,6 +74,6 @@
       </geometry>
     </visual>
-   <!-- arm left -->
-    <collision name="caster_back_collision">
+   <!-- arm right -->
+    <collision name="arm_right_collision">
       <origin rpy=" 0 0 0" xyz="0.1 0.20 0.05"/>
       <geometry>
@@ -107,5 +81,5 @@
       </geometry>
     </collision>
-    <visual name="caster_back_visual">
+    <visual name="arm_right_visual">
       <origin rpy=" 0 0 0" xyz="0.1 0.20 0.05"/>
       <geometry>
@@ -114,5 +88,72 @@
     </visual>
   </link>
-   <link name="link_right_wheel">
+<!-- castor wheels -->
+ <link name="link_castor_axis">
+    <!-- pose and inertial -->
+    <pose>0 0 0.1 0 0 0</pose>
+    <xacro:default_inertial mass="2" />
+    <!-- body -->
+    <collision name="collision_chassis">
+      <origin rpy="0 0 0" xyz="0.025 0 0"/>
+      <geometry>
+        <box size="0.05 0.035 0.03"/>
+      </geometry>
+    </collision>
+    <visual>
+      <origin rpy="0 0 0" xyz="-0.025 0 0"/>
+      <geometry>
+        <box size="0.05 0.035 0.03"/>
+      </geometry>
+    </visual>
+  </link>
+  <link name="link_castor_wheel">
+    <xacro:default_inertial mass="0.8"/>
+    <collision name="link_castor_wheel_collision">
+      <origin rpy="0 1.5707 1.5707" xyz="0 0 0"/>
+      <geometry>
+        <cylinder length="0.02" radius="0.03"/>
+      </geometry>
+    </collision>
+    <visual name="link_castor_wheel_visual">
+      <origin rpy="0 1.5707 1.5707" xyz="0 0 0"/>
+      <geometry>
+        <cylinder length="0.02" radius="0.03"/>
+      </geometry>
+    </visual>
+  </link>
+  <joint name="joint_castor_wheel" type="continuous">
+    <origin rpy="0 0 0" xyz="0.05 0 -0.015"/>
+    <child link="link_castor_wheel"/>
+    <parent link="link_castor_axis"/>
+    <axis rpy="0 0 0" xyz="0 1 0"/>
+    <limit effort="10000" velocity="1000"/>
+    <joint_properties damping="1.0" friction="1.0"/>
+  </joint>
+  <joint name="joint_castor_axis" type="continuous">
+    <origin rpy="0 0 0" xyz="0.1 0 -0.20"/>
+    <child link="link_castor_axis"/>
+    <parent link="link_chassis"/>
+    <axis rpy="0 0 0" xyz="0 0 1"/>
+    <limit effort="10000" velocity="1000"/>
+    <joint_properties damping="1.0" friction="1.0"/>
+  </joint>
+ <!-- Main wheels -->
+  <joint name="joint_right_wheel" type="continuous">
+    <origin rpy="0 0 0" xyz="-0.1 0.175 -0.14"/>
+    <child link="link_right_wheel"/>
+    <parent link="link_chassis"/>
+    <axis rpy="0 0 0" xyz="0 1 0"/>
+    <limit effort="10000" velocity="1000"/>
+    <joint_properties damping="1.0" friction="1.0"/>
+  </joint>
+  <joint name="joint_left_wheel" type="continuous">
+    <origin rpy="0 0 0" xyz="-0.1 -0.175 -0.14"/>
+    <child link="link_left_wheel"/>
+    <parent link="link_chassis"/>
+    <axis rpy="0 0 0" xyz="0 1 0"/>
+    <limit effort="10000" velocity="1000"/>
+    <joint_properties damping="1.0" friction="1.0"/>
+  </joint>
+  <link name="link_right_wheel">
     <xacro:default_inertial mass="0.2"/>
     <collision name="link_right_wheel_collision">
@@ -138,20 +179,5 @@
     </visual>
   </link>
-  <joint name="joint_right_wheel" type="continuous">
-    <origin rpy="0 0 0" xyz="0 0.175 -0.15"/>
-    <child link="link_right_wheel"/>
-    <parent link="link_chassis"/>
-    <axis rpy="0 0 0" xyz="0 1 0"/>
-    <limit effort="10000" velocity="1000"/>
-    <joint_properties damping="1.0" friction="1.0"/>
-  </joint>
-  <joint name="joint_left_wheel" type="continuous">
-    <origin rpy="0 0 0" xyz="0 -0.175 -0.15"/>
-    <child link="link_left_wheel"/>
-    <parent link="link_chassis"/>
-    <axis rpy="0 0 0" xyz="0 1 0"/>
-    <limit effort="10000" velocity="1000"/>
-    <joint_properties damping="1.0" friction="1.0"/>
-  </joint>
+<!-- Neck and head -->
   <link name="neck_link">
 	    <collision>
@@ -197,5 +223,5 @@
 	      <mass value="1e-5" />
 	      <origin xyz="0 0 0" rpy="0 0 0"/>
-	      <inertia ixx="1e-6" ixy="0" ixz="0" iyy="1e-6" iyz="0" izz="1e-6" />
+	      <inertia ixx="1e-6" ixy="0" ixz="0" iyy="1" iyz="0" izz="1e-6" />
 	    </inertial>
   </link>

Commit message: Explore + testing
The explore-lite node have been added to the workspace and some other little modification to adjust the robot behavior during testing of the explore feature

File: urdf/Pet/robot.xacro (robot description, xacro)
@@ -131,5 +131,5 @@
   </joint>
   <joint name="joint_castor_axis" type="continuous">
-    <origin rpy="0 0 0" xyz="0.1 0 -0.20"/>
+    <origin rpy="0 0 0" xyz="0.18 0 -0.20"/>
     <child link="link_castor_axis"/>
     <parent link="link_chassis"/>
